File: butler/version-0/butler.kicad_pcb (KiCad board)
At the start: 2 copper layers, 46.2 x 49.8 mm, 40 parts, among them J1 CONN_01X01, J2 CONN_01X01, J3 CONN_01X01, J4 CONN_01X01, P1 CONN_BATT/MOT, P2 CONN_SW, P3 CONN_SERIAL, Q1 P/N_MOS, Q2 P/N_MOS, U1 WeMos_mini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

Commit message: updated library names after lib refactoring
Parts:
- U1: footprint wemos-d1-mini:wemos-d1-mini -> wemos-d1-mini:wemos-d1-mini-with-pin-header-and-connector
