File: butler/version-0.2-prototyping-pcb/butler.kicad_pcb (KiCad board)
At the start: 2 copper layers, 160 x 100.3 mm, 58 parts, among them J1 CONN_01X01, J10 TX, J11 SWITCH_A, J12 SWITCH_B, J13 GND, J14 SW_V+, J15 SER_3V3, J16 GND, J17 1W, J18 SDA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

Commit message: minor change to satisfy DRC
Routing:
- net /BATT+: track 295.9 -> 309.9 mm
- net /SW_B: track 69.4 -> 80.9 mm
- net VCC: track 114.1 -> 121.7 mm
Changed lines of the file:
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@@
   (general
     (links 118)
-    (no_connects 2)
+    (no_connects 0)
     (area 25.299999 25.299999 185.520001 125.830001)
     (thickness 1.6)
     (drawings 9)
-    (tracks 445)
+    (tracks 450)
     (zones 0)
     (modules 58)
@@
   (segment (start 33.02 33.02) (end 36.219999 29.820001) (width 1.016) (layer F.Cu) (net 1))
   (segment (start 174.600001 29.820001) (end 177.8 33.02) (width 1.016) (layer F.Cu) (net 1))
+  (segment (start 91.44 73.66) (end 83.312 65.532) (width 1.016) (layer B.Cu) (net 2))
+  (segment (start 87.900001 42.147999) (end 100.346005 42.147999) (width 1.016) (layer B.Cu) (net 2))
+  (segment (start 83.312 65.532) (end 83.312 46.736) (width 1.016) (layer B.Cu) (net 2))
+  (segment (start 100.346005 42.147999) (end 101.346004 41.148) (width 1.016) (layer B.Cu) (net 2))
+  (segment (start 83.312 46.736) (end 87.900001 42.147999) (width 1.016) (layer B.Cu) (net 2))
   (segment (start 101.346 38.247598) (end 101.346004 38.247602) (width 1.016) (layer F.Cu) (net 2))
   (segment (start 101.346004 38.247602) (end 101.346004 41.148) (width 1.016) (layer F.Cu) (net 2))
@@
   (segment (start 86.106 73.66) (end 91.44 73.66) (width 1.016) (layer F.Cu) (net 2))
   (via (at 101.346004 41.148) (size 2) (drill 0) (layers F.Cu B.Cu) (net 2))
-  (segment (start 91.44 51.054004) (end 100.346005 42.147999) (width 1.016) (layer B.Cu) (net 2))
-  (segment (start 91.44 73.66) (end 91.44 51.054004) (width 1.016) (layer B.Cu) (net 2))
-  (segment (start 100.346005 42.147999) (end 101.346004 41.148) (width 1.016) (layer B.Cu) (net 2))
   (segment (start 60.96 44.45) (end 60.96 33.274) (width 1.016) (layer F.Cu) (net 2))
   (segment (start 60.96 33.274) (end 62.484 31.75) (width 1.016) (layer F.Cu) (net 2))
@@
   (segment (start 59.396 38.1) (end 60.96 39.664) (width 1.016) (layer F.Cu) (net 2))
   (segment (start 60.96 39.664) (end 60.96 44.45) (width 1.016) (layer F.Cu) (net 2))
+  (segment (start 88.9 55.88) (end 96.52 55.88) (width 1.016) (layer B.Cu) (net 3))
   (segment (start 96.52 57.294213) (end 96.52 55.88) (width 1.016) (layer F.Cu) (net 3))
   (segment (start 100.837992 67.564) (end 96.52 63.246008) (width 1.016) (layer F.Cu) (net 3))
@@
   (segment (start 108.458 72.39) (end 90.598 90.25) (width 1.016) (layer F.Cu) (net 8))
   (segment (start 90.598 90.25) (end 86.36 90.25) (width 1.016) (layer F.Cu) (net 8))
+  (segment (start 88.9 60.96) (end 90.314213 60.96) (width 1.016) (layer B.Cu) (net 9))
+  (segment (start 90.314213 60.96) (end 100.33 60.96) (width 1.016) (layer B.Cu) (net 9))
   (segment (start 87.485787 60.96) (end 88.9 60.96) (width 1.016) (layer F.Cu) (net 9))
   (segment (start 86.626391 60.96) (end 87.485787 60.96) (width 1.016) (layer F.Cu) (net 9))
